File: MainModule/Hardware/MainModule.sch (EAGLE design)
At the start: 0 parts

Commit message: start of design
Parts:
- added LPC1: (no value), LPCXpresso_LPC1769:LPCXPRESSO_LPC1769
- added U1, U2, U3: ULN2803ADW, ULN2803:ULN2803ADW
- added X1, X2, X3: MKDSN1,5/8-5,08, con-phoenix-508:MKDSN1,5/8-5,08
- added X4: MKDSN1,5/2-5,08, con-phoenix-508:MKDSN1,5/2-5,08
- added X5: MKDSN1,5/3-5,08, con-phoenix-508:MKDSN1,5/3-5,08
Connections:
- new net GND: U1.GND, U2.GND, U3.GND
- new net N$1: LPC1.5, U1.1B
- new net N$10: LPC1.14, U2.2B
- new net N$11: LPC1.15, U2.3B
- new net N$12: LPC1.16, U2.4B
- new net N$13: LPC1.17, U2.5B
- new net N$14: LPC1.18, U2.6B
- new net N$15: LPC1.19, U2.7B
- new net N$16: LPC1.20, U2.8B
- new net N$17: LPC1.38, U3.8B
- new net N$18: LPC1.39, U3.7B
- new net N$19: LPC1.48, U3.6B
- new net N$2: LPC1.6, U1.2B
- new net N$20: LPC1.49, U3.5B
- new net N$21: LPC1.50, U3.4B
- new net N$22: LPC1.73, U3.3B
- new net N$23: LPC1.72, U3.2B
- new net N$24: LPC1.71, U3.1B
- new net N$25: U1.1C, X1-1.KL
- new net N$26: U1.2C, X1-2.KL
- new net N$27: U1.3C, X1-3.KL
- new net N$28: U1.4C, X1-4.KL
- new net N$29: U1.5C, X1-5.KL
- new net N$3: LPC1.7, U1.3B
- new net N$30: U1.6C, X1-6.KL
- new net N$31: U1.7C, X1-7.KL
- new net N$32: U1.8C, X1-8.KL
- new net N$33: U2.1C, X2-1.KL
- new net N$34: U2.2C, X2-2.KL
- new net N$35: U2.3C, X2-3.KL
- new net N$36: U2.4C, X2-4.KL
- new net N$37: U2.5C, X2-5.KL
- new net N$38: U2.6C, X2-6.KL
- new net N$39: U2.7C, X2-7.KL
- new net N$4: LPC1.8, U1.4B
- new net N$40: U2.8C, X2-8.KL
- new net N$41: U3.1C, X3-1.KL
- new net N$42: U3.2C, X3-2.KL
- new net N$43: U3.3C, X3-3.KL
- new net N$44: U3.4C, X3-4.KL
- new net N$45: U3.5C, X3-5.KL
- new net N$46: U3.6C, X3-6.KL
- new net N$47: U3.7C, X3-7.KL
- new net N$48: U3.8C, X3-8.KL
- new net N$5: LPC1.9, U1.5B
- new net N$6: LPC1.10, U1.6B
- new net N$7: LPC1.11, U1.7B
- new net N$8: LPC1.12, U1.8B
- new net N$9: LPC1.13, U2.1B
